File: hardware/KiCad/OpenMI/Sensing.kicad_sch (KiCad schematic)
At the start: 60 parts, among them U10 MCS1802GS-05, U11 MCP6001T-OT, U12 MCP6567-SN, U14 MCP6561-OT, U2 INA381A2IDGS, U5 MCP6004-SL, U7 MCP6001T-OT

Commit message: feat(hw): Adds PV module voltage and current sensing (#3)
* Adds first draft of pv-panel voltage and current sensing.

* Adds specific values for sense resistors.

* Set anti-aliasing cutoff frequency to 4.8kHz.
Adds documentation.

* Adds ADE7912

* Tidy up schematics. Adds sheet symbols to root.

* updates symbols from library.

* chore: 🤖 KiCad export

---------

Co-authored-by: github-actions <41898282+github-actions[bot]@users.noreply.github.com>
Parts:
- R11, R13, R42, R45: OC_LCSC (none) -> C25804
- R46: OC_MOUSER (none) -> 667-ERJ-C1CFR02U
Changed lines of the file:
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@@
+      (effects (font (size 1.27 1.27)) hide)
+    )
+    (property "OC_LCSC" "C25804" (at 200.66 55.88 0)
       (effects (font (size 1.27 1.27)) hide)
     )
@@
       (effects (font (size 1.27 1.27)) hide)
     )
+    (property "OC_LCSC" "C25804" (at 96.52 171.45 0)
+      (effects (font (size 1.27 1.27)) hide)
+    )
     (pin "1")
     (pin "2")
@@
       (effects (font (size 1.27 1.27)) hide)
     )
+    (property "OC_LCSC" "C25804" (at 220.98 77.47 0)
+      (effects (font (size 1.27 1.27)) hide)
+    )
     (pin "1")
     (pin "2")
@@
       (effects (font (size 1.27 1.27)) hide)
     )
-    (property "OC_MOUSER" "" (at 40.64 116.84 0)
+    (property "OC_MOUSER" "667-ERJ-C1CFR02U" (at 40.64 116.84 0)
       (effects (font (size 1.27 1.27)) hide)
     )
@@
     )
   )
-  (symbol (lib_name "10K_1") (lib_id "_R_0603:10K") (at 107.95 71.12 0) (unit 1)
+  (symbol (lib_id "_R_0603:10K") (at 107.95 71.12 0) (unit 1)
     (in_bom yes) (on_board yes) (dnp no) (fields_autoplaced)
     (property "Reference" "R53" (at 110.49 70.485 0)
@@
     )
     (property "OC_REICHELT" "" (at 127 142.24 0)
+      (effects (font (size 1.27 1.27)) hide)
+    )
+    (property "OC_LCSC" "C25804" (at 127 142.24 0)
       (effects (font (size 1.27 1.27)) hide)
     )
@@
     )
   )
-  (symbol (lib_name "10K_1") (lib_id "_R_0603:10K") (at 64.77 68.58 0) (unit 1)
+  (symbol (lib_id "_R_0603:10K") (at 64.77 68.58 0) (unit 1)
     (in_bom yes) (on_board yes) (dnp no) (fields_autoplaced)
     (property "Reference" "R55" (at 67.31 67.945 0)
@@
     )
   )
-  (symbol (lib_name "10K_1") (lib_id "_R_0603:10K") (at 64.77 83.82 0) (unit 1)
+  (symbol (lib_id "_R_0603:10K") (at 64.77 83.82 0) (unit 1)
     (in_bom yes) (on_board yes) (dnp no) (fields_autoplaced)
     (property "Reference" "R56" (at 67.31 83.185 0)
